File: ESP32_Sharonov_test_board/KiCad/ESP32_Sharonov_test_board/ESP32-WROOM-32.kicad_sch (KiCad schematic)
At the start: 0 parts

Commit message: ..
Changed lines of the file:
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@@
+    (effects (font (size 1.27 1.27)) (justify left))
+  )
+  (hierarchical_label "16 IO13" (shape bidirectional) (at 87.63 109.22 0) (fields_autoplaced)
     (effects (font (size 1.27 1.27)) (justify left))
   )
@@
     (effects (font (size 1.27 1.27)) (justify left))
   )
+  (hierarchical_label "27 IO16 RX2" (shape input) (at 191.77 105.41 0) (fields_autoplaced)
+    (effects (font (size 1.27 1.27)) (justify left))
+  )
   (hierarchical_label "25 IO0 (boot)" (shape input) (at 191.77 120.65 0) (fields_autoplaced)
+    (effects (font (size 1.27 1.27)) (justify left))
+  )
+  (hierarchical_label "28 IO17 TX2" (shape output) (at 191.77 101.6 0) (fields_autoplaced)
     (effects (font (size 1.27 1.27)) (justify left))
   )
@@
     (effects (font (size 1.27 1.27)) (justify left))
   )
+  (hierarchical_label "33 IO21" (shape bidirectional) (at 87.63 106.68 0) (fields_autoplaced)
+    (effects (font (size 1.27 1.27)) (justify left))
+  )
   (hierarchical_label "35 TXD0" (shape output) (at 191.77 80.01 0) (fields_autoplaced)
     (effects (font (size 1.27 1.27)) (justify left))
   )
-  (hierarchical_label "27 IO16" (shape bidirectional) (at 87.63 105.41 0) (fields_autoplaced)
+  (hierarchical_label "9 IO33" (shape bidirectional) (at 87.63 124.46 0) (fields_autoplaced)
     (effects (font (size 1.27 1.27)) (justify left))
   )
-  (hierarchical_label "9 IO33" (shape bidirectional) (at 87.63 124.46 0) (fields_autoplaced)
+  (hierarchical_label "37 IO23" (shape bidirectional) (at 87.63 101.6 0) (fields_autoplaced)
     (effects (font (size 1.27 1.27)) (justify left))
   )
@@
     (effects (font (size 1.27 1.27)) (justify left))
   )
-  (hierarchical_label "28 IO17" (shape bidirectional) (at 87.63 109.22 0) (fields_autoplaced)
+  (hierarchical_label "36 IO22" (shape bidirectional) (at 87.63 104.14 0) (fields_autoplaced)
     (effects (font (size 1.27 1.27)) (justify left))
   )
