File: ESP32_Sharonov_test_board/KiCad/ESP32_Sharonov_test_board/ESP32-WROOM-32.kicad_sch (KiCad schematic)
At the start: 0 parts

Commit message: ...
Changed lines of the file:
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@@
+    (effects (font (size 1.27 1.27)) (justify left))
+  )
+  (hierarchical_label "8 IO35" (shape input) (at 191.77 104.14 0) (fields_autoplaced)
     (effects (font (size 1.27 1.27)) (justify left))
   )
@@
     (effects (font (size 1.27 1.27)) (justify left))
   )
+  (hierarchical_label "7 IO34" (shape input) (at 191.77 101.6 0) (fields_autoplaced)
+    (effects (font (size 1.27 1.27)) (justify left))
+  )

Commit message: ююю
Changed lines of the file:
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@@
+    (effects (font (size 1.27 1.27)) (justify left))
+  )
+  (hierarchical_label "3 EN" (shape input) (at 87.63 67.31 0) (fields_autoplaced)
     (effects (font (size 1.27 1.27)) (justify left))
   )
