File: ESP32_Sharonov_test_board/KiCad/ESP32_Sharonov_test_board/ESP32_Sharonov_test_board.kicad_sch (KiCad schematic)
At the start: 11 parts, among them J1 ESP-UART, J2 AUX32, J3 AUX33, J4 AUX16, J5 AUX17, J6 AUX18, J7 AUX19

Commit message: ..
Parts:
- removed J4: AUX16, symbol Connector:Conn_01x01_Pin
- removed J5: AUX17, symbol Connector:Conn_01x01_Pin
Other:
- sheet ESP32-WROOM-32 ports: added 16 IO13, 27 IO16 RX2, 28 IO17 TX2, 33 IO21, 36 IO22, 37 IO23; removed 27 IO16, 28 IO17
- note added: "Можно использовать, как двунаправленные без ограничений: IO18,19 IO32,33 IO13 IO21,22,23 Занятые: IO4 - OLED-VCC IO25,26,27 - Энкодер IO16,17 - SA818-UART"
- note removed: "Можно использовать, как двунаправленные без ограничений: IO16,17,18,19 IO32,33 IO4 - OLED+ IO25,26,27 - Энкодер Ещё есть под JTAG но их на всякий случай лучше не занимать"
- moved on the sheet: J2, J3, J6, J7
