File: ESP32_Sharonov_test_board/KiCad/ESP32_Sharonov_test_board/ESP32_Sharonov_test_board.kicad_sch (KiCad schematic)
At the start: 11 parts, among them J1 ESP-UART, J2 AUX32, J3 AUX33, J4 AUX16, J5 AUX17, J6 AUX18, J7 AUX19

Commit message: ...
Parts:
- removed J4: AUX16, symbol Connector:Conn_01x01_Pin
- removed J7: AUX19, symbol Connector:Conn_01x01_Pin
- J5: value AUX17 -> AUX34
- J6: value AUX18 -> AUX35
Connections:
- net ESP32-WROOM-32/28 IO17: no longer J5.1 (Pin_1)
- net ESP32-WROOM-32/30 IO18: no longer J6.1 (Pin_1)
- new net ESP32-WROOM-32/7 IO34: J5.1 (Pin_1)
- new net ESP32-WROOM-32/8 IO35: J6.1 (Pin_1)
Other:
- added sheet SA818S (SA818S.kicad_sch)
- sheet ESP32-WROOM-32 ports: added 7 IO34, 8 IO35; removed none
- note added: "RX2"
- note added: "TX2"
- note added: "Можно использовать, как двунаправленные без ограничений: IO32,33 Занятые: IO16,17,18,19 - SA818S IO4 - OLED+ IO25,26,27 - Энкодер только,как входы: (и нет pullup) IO34,35,36,39"
- note added: "Осталось развести земли и питания и надо сделать контакные площадки для оставшихся портов (AUX...) без отверстий (чтобы можно было подпаять провода при необходимости)."
- note added: "здесь не все ноги указаны!"
- note removed: "Можно использовать, как двунаправленные без ограничений: IO16,17,18,19 IO32,33 IO4 - OLED+ IO25,26,27 - Энкодер Ещё есть под JTAG но их на всякий случай лучше не занимать"
- note removed: "Осталось развести земли и питания и надо сделать контакные площадки для оставшихся портов без отверстий (чтобы можно было подпаять провода при необходимости). Для подключения датчиков/исполнительных механизмов (AUX...)"
- moved on the sheet: J2, J3

Commit message: ....
Connections:
- net ESP32-WROOM-32/30 IO18: now also J2.1 (Pin_1)
- net ESP32-WROOM-32/8 IO32: no longer J2.1 (Pin_1)
Other:
- note added: "сюда только пин с ADC"
Changed lines of the file:
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@@
+    (stroke (width 0) (type default))
+  )
+  (wire (pts (xy 185.42 96.52) (xy 245.11 96.52))
     (stroke (width 0) (type default))
   )
@@
     (stroke (width 0) (type default))
   )
+  (wire (pts (xy 158.75 97.79) (xy 157.48 97.79))
+    (stroke (width 0) (type default))
+  )
   (wire (pts (xy 158.75 85.09) (xy 104.14 85.09))
     (stroke (width 0) (type default))
@@
     (stroke (width 0) (type default))
   )
-  (wire (pts (xy 158.75 99.06) (xy 157.48 99.06))
-    (stroke (width 0) (type default))
-  )
   (wire (pts (xy 157.48 96.52) (xy 152.4 96.52))
     (stroke (width 0) (type default))
@@
     (stroke (width 0) (type default))
   )
-  (wire (pts (xy 185.42 96.52) (xy 245.11 96.52))
-    (stroke (width 0) (type default))
-  )
   (wire (pts (xy 158.75 81.28) (xy 123.19 81.28))
     (stroke (width 0) (type default))
@@
     (stroke (width 0) (type default))
   )
-  (wire (pts (xy 157.48 99.06) (xy 157.48 96.52))
-    (stroke (width 0) (type default))
-  )
   (wire (pts (xy 95.25 85.09) (xy 95.25 87.63))
     (stroke (width 0) (type default))
@@
     (stroke (width 0) (type default))
   )
+  (wire (pts (xy 157.48 97.79) (xy 157.48 96.52))
+    (stroke (width 0) (type default))
+  )
   (wire (pts (xy 204.47 54.61) (xy 191.77 54.61))
     (stroke (width 0) (type default))
@@
   (wire (pts (xy 111.76 57.15) (xy 111.76 58.42))
     (stroke (width 0) (type default))
+  )
+  (text "сюда только пин с ADC" (at 185.42 96.52 0)
+    (effects (font (size 1.27 1.27)) (justify left bottom))
   )
   (text "здесь\nне\nвсе\nноги\nуказаны!" (at 167.64 80.01 0)
@@
       (effects (font (size 1.27 1.27)) (justify left))
     )
-    (pin "8 IO32" bidirectional (at 158.75 99.06 180)
-      (effects (font (size 1.27 1.27)) (justify left))
+    (pin "8 IO32" bidirectional (at 185.42 96.52 0)
+      (effects (font (size 1.27 1.27)) (justify right))
     )
     (pin "9 IO33" bidirectional (at 158.75 102.87 180)
@@
       (effects (font (size 1.27 1.27)) (justify right))
     )
-    (pin "30 IO18" bidirectional (at 185.42 96.52 0)
-      (effects (font (size 1.27 1.27)) (justify right))
+    (pin "30 IO18" bidirectional (at 158.75 97.79 180)
+      (effects (font (size 1.27 1.27)) (justify left))
     )
     (pin "31 IO19" bidirectional (at 185.42 101.6 0)

Commit message: ююю
Other:
- note added: "Можно использовать, как двунаправленные без ограничений: IO18,33 Занятые: IO16,17,19,32 - SA818S IO4 - OLED+ IO25,26,27 - Энкодер только,как входы: (и нет pullup) IO34,35,36,39"
- note removed: "Можно использовать, как двунаправленные без ограничений: IO32,33 Занятые: IO16,17,18,19 - SA818S IO4 - OLED+ IO25,26,27 - Энкодер только,как входы: (и нет pullup) IO34,35,36,39"
Changed lines of the file:
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@@
     (effects (font (size 1.27 1.27)) (justify left bottom))
   )
-  (text "Можно использовать, как \nдвунаправленные без ограничений:\nIO32,33\n\nЗанятые:\nIO16,17,18,19 - SA818S\nIO4 - OLED+\nIO25,26,27 - Энкодер\n\nтолько,как входы:\n(и нет pullup)\nIO34,35,36,39 \n\n\n"
+  (text "Можно использовать, как \nдвунаправленные без ограничений:\nIO18,33\n\nЗанятые:\nIO16,17,19,32 - SA818S\nIO4 - OLED+\nIO25,26,27 - Энкодер\n\nтолько,как входы:\n(и нет pullup)\nIO34,35,36,39 \n\n\n"
     (at 160.02 156.21 0)
     (effects (font (size 1.27 1.27)) (justify left bottom))

Commit message: ююю
Parts:
- removed J5: AUX34, symbol Connector:Conn_01x01_Pin
Other:
- sheet SA818S ports: added EN_V1 (audio on); removed none
- note added: "Можно использовать, как двунаправленные без ограничений: IO18,33 из них занятые: IO16,17,19,32 - SA818S IO4 - OLED+ IO25,26,27 - Энкодер только,как входы: (и нет pullup) IO35,36,39 из них занятые: IO34 - SA818S"
- note removed: "Можно использовать, как двунаправленные без ограничений: IO18,33 Занятые: IO16,17,19,32 - SA818S IO4 - OLED+ IO25,26,27 - Энкодер только,как входы: (и нет pullup) IO34,35,36,39"
Changed lines of the file:
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@@
+    (stroke (width 0) (type default))
+  )
+  (wire (pts (xy 185.42 104.14) (xy 245.11 104.14))
     (stroke (width 0) (type default))
   )
@@
     (stroke (width 0) (type default))
   )
-  (wire (pts (xy 152.4 106.68) (xy 152.4 107.95))
-    (stroke (width 0) (type default))
-  )
   (wire (pts (xy 156.21 102.87) (xy 156.21 100.33))
     (stroke (width 0) (type default))
@@
     (stroke (width 0) (type default))
   )
-  (wire (pts (xy 158.75 106.68) (xy 152.4 106.68))
-    (stroke (width 0) (type default))
-  )
   (wire (pts (xy 157.48 97.79) (xy 157.48 96.52))
     (stroke (width 0) (type default))
@@
     (effects (font (size 1.27 1.27)) (justify left bottom))
   )
-  (text "Можно использовать, как \nдвунаправленные без ограничений:\nIO18,33\n\nЗанятые:\nIO16,17,19,32 - SA818S\nIO4 - OLED+\nIO25,26,27 - Энкодер\n\nтолько,как входы:\n(и нет pullup)\nIO34,35,36,39 \n\n\n"
-    (at 160.02 156.21 0)
+  (text "Можно использовать, как \nдвунаправленные без ограничений:\nIO18,33\n\nиз них занятые:\nIO16,17,19,32 - SA818S\nIO4 - OLED+\nIO25,26,27 - Энкодер\n\nтолько,как входы:\n(и нет pullup)\nIO35,36,39 \n\nиз них занятые:\nIO34 - SA818S\n\n\n"
+    (at 157.48 162.56 0)
     (effects (font (size 1.27 1.27)) (justify left bottom))
   )
@@
   )
   (text "Для прошивки через UART:\nУстановить джампер на 1-2,\nподать питание.\nЗалить прошивку.\nВернуть джампер на 2-3"
-    (at 207.01 115.57 0)
+    (at 208.28 119.38 0)
     (effects (font (size 1.27 1.27)) (justify left bottom))
   )
@@
         (path "/03a54034-ff9b-422a-870f-6d595fbb611a"
           (reference "#PWR01") (unit 1)
-        )
-      )
-    )
-  )
-  (symbol (lib_id "Connector:Conn_01x01_Pin") (at 147.32 107.95 0) (unit 1)
-    (in_bom yes) (on_board yes) (dnp no) (fields_autoplaced)
-    (property "Reference" "J5" (at 147.955 102.87 0)
-      (effects (font (size 1.27 1.27)))
-    )
-    (property "Value" "AUX34" (at 147.955 105.41 0)
-      (effects (font (size 1.27 1.27)))
-    )
-    (property "Footprint" "" (at 147.32 107.95 0)
-      (effects (font (size 1.27 1.27)) hide)
-    )
-    (property "Datasheet" "~" (at 147.32 107.95 0)
-      (effects (font (size 1.27 1.27)) hide)
-    )
-    (pin "1")
-    (instances
-      (project "ESP32_Sharonov_test_board"
-        (path "/03a54034-ff9b-422a-870f-6d595fbb611a"
-          (reference "J5") (unit 1)
         )
       )
@@
       (effects (font (size 1.27 1.27)) (justify right))
     )
-    (pin "7 IO34" input (at 158.75 106.68 180)
-      (effects (font (size 1.27 1.27)) (justify left))
+    (pin "7 IO34" input (at 185.42 104.14 0)
+      (effects (font (size 1.27 1.27)) (justify right))
     )
     (pin "8 IO35" input (at 158.75 110.49 180)
@@
       (effects (font (size 1.27 1.27)) (justify left))
     )
+    (pin "EN_V1 (audio on)" output (at 245.11 104.14 180)
+      (effects (font (size 1.27 1.27)) (justify left))
+    )

Commit message: ююю
Other:
- sheet ESP32-WROOM-32 ports: added 3 EN; removed none
Changed lines of the file:
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@@
+    (stroke (width 0) (type default))
+  )
+  (wire (pts (xy 158.75 73.66) (xy 139.7 73.66))
     (stroke (width 0) (type default))
   )
@@
   )
   (wire (pts (xy 185.42 114.3) (xy 190.5 114.3))
+    (stroke (width 0) (type default))
+  )
+  (wire (pts (xy 139.7 73.66) (xy 139.7 58.42))
     (stroke (width 0) (type default))
   )
@@
         (path "/03a54034-ff9b-422a-870f-6d595fbb611a"
           (reference "#PWR04") (unit 1)
+        )
+      )
+    )
+  )
+  (symbol (lib_id "power:+3.3V") (at 139.7 58.42 0) (unit 1)
+    (in_bom yes) (on_board yes) (dnp no) (fields_autoplaced)
+    (property "Reference" "#PWR06" (at 139.7 62.23 0)
+      (effects (font (size 1.27 1.27)) hide)
+    )
+    (property "Value" "+3.3V" (at 139.7 53.34 0)
+      (effects (font (size 1.27 1.27)))
+    )
+    (property "Footprint" "" (at 139.7 58.42 0)
+      (effects (font (size 1.27 1.27)) hide)
+    )
+    (property "Datasheet" "" (at 139.7 58.42 0)
+      (effects (font (size 1.27 1.27)) hide)
+    )
+    (pin "1")
+    (instances
+      (project "ESP32_Sharonov_test_board"
+        (path "/03a54034-ff9b-422a-870f-6d595fbb611a"
+          (reference "#PWR06") (unit 1)
         )
       )
@@
       (effects (font (size 1.27 1.27)) (justify left))
     )
+    (pin "3 EN" input (at 158.75 73.66 180)
+      (effects (font (size 1.27 1.27)) (justify left))
+    )
