File: ESP32_Sharonov_test_board/KiCad/ESP32_Sharonov_test_board/SA818S.kicad_sch (KiCad schematic)
At the start: 0 parts

Commit message: ююю
Changed lines of the file:
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@@
 (kicad_sch (version 20230121) (generator eeschema)
   (paper "A4")
+  (hierarchical_label "EN_V1 (audio on)" (shape output) (at 124.46 96.52 0) (fields_autoplaced)
+    (effects (font (size 1.27 1.27)) (justify left))
+  )
   (hierarchical_label "TX (uart)" (shape output) (at 125.73 83.82 0) (fields_autoplaced)
     (effects (font (size 1.27 1.27)) (justify left))
